Commit message: Add R2400 3D models

File: src/pf_description/urdf/r2400.urdf.xacro (robot description, xacro)
@@ -6,5 +6,5 @@
                 <origin xyz="0 0 0" rpy="0 0 0" />
                 <geometry>
-                    <mesh filename="package://pf_description/meshes/R2000.stl" scale="0.001 0.001 0.001" />
+                    <mesh filename="package://pf_description/meshes/R2400.stl" scale="0.001 0.001 0.001" />
                 </geometry>
             </visual>
